File: hardware/speedy_bldc.sch (EAGLE design)
At the start: 153 parts, among them IC1 STM32F40X, J2 Throttle, J4 Brake, U1 MCP2551, X1 X1

Commit message: Added BOM
Parts:
- removed TP1, TP10, TP12, TP2, TP4, TP5, TP7, TP8: TPB1,27, testpad:TPB1,27
- added C49, C50, C51: 100n, SparkFun-Capacitors:CAP0603-CAP
- added D6: (no value), SparkFun-LED:LED-FKIT-1206
- added PT1: 2PT_GND_TIE, SparkFun-Passives:2PT_GND_TIE
- added R37: 100R, SparkFun-Resistors:RESISTOR0603
- C1, C2, C30: PARTNO (none) -> 399-7880-1-ND
- C10, C11, C13, C18, C21, C3, C4, C5: PARTNO (none) -> 399-7845-1-ND
- C12: PARTNO (none) -> 587-1097-1-ND
- C14, C15, C16: PARTNO (none) -> 445-5208-1-ND
- C17: DIGIKEY 490-3907-1-ND -> (none); PARTNO (none) -> 490-3907-1-ND
- C19, C20: value 10u -> 4.7u; PARTNO (none) -> 1276-1248-1-ND
- C22, C23, C24, C25, C26, C28, C31: PARTNO (none) -> 587-3248-1-ND
- C27, C7: device SparkFun-Capacitors:CAP0805 -> SparkFun-Capacitors:CAP0603-CAP; PARTNO (none) -> 1276-1879-1-ND
- C29: PARTNO (none) -> 712-1345-1-ND
- C32, C33, C34, C35: PARTNO (none) -> 493-11950-1-ND
- C36, C48: PARTNO (none) -> 399-1097-1-ND
- C37, C38: PARTNO (none) -> 712-1318-1-ND
- C39, C40, C41, C42, C43, C44, C45, C46: PARTNO (none) -> 1276-1879-1-ND
- C47: PARTNO (none) -> 490-3302-1-ND
- C6: PARTNO (none) -> 1276-1936-1-ND
- C8: device SparkFun-Capacitors:CAP0805 -> SparkFun-Capacitors:CAP0603-CAP; PARTNO (none) -> 587-2984-1-ND
- C9: PARTNO (none) -> 587-2984-1-ND
- D1: value (none) -> SCHOTTKY_SMA; device diode:SCHOTTKY-DIODESMC -> speedy_bldc:SCHOTTKY_SMA; DIGIKEY VS-30BQ100-M3/9AT-ND -> (none); PARTNO (none) -> 497-12285-1-ND
- D2, D3, D4, D5: PARTNO (none) -> 160-1457-1-ND
- IC1: DIGIKEY 497-11767-ND -> (none); PARTNO (none) -> 497-11767-ND
- JP2: PARTNO (none) -> A33210-ND
- L1: DIGIKEY 490-5272-1-ND -> (none); PARTNO (none) -> 490-5272-1-ND
- R1, R2, R3, R4, R5, R6: PARTNO (none) -> 1276-4991-1-ND
- R10, R7, R8, R9: PARTNO (none) -> 311-100HRCT-ND
- R11, R12, R13, R14, R15, R36: PARTNO (none) -> 311-10KGRCT-ND
- R16: value 31.6 -> 31.6K; PARTNO (none) -> 311-31.6KHRCT-ND
- R17: PARTNO (none) -> 541-205KHCT-ND
- R18: PARTNO (none) -> 311-28.0KHRCT-ND
- R19, R20, R21: PARTNO (none) -> 311-680HRCT-ND
- R22, R26, R28, R30: PARTNO (none) -> 311-39.0KHRCT-ND
- R23, R27, R29, R31: PARTNO (none) -> 311-2.20KHRCT-ND
- R24, R25, R33, R34: value 680R -> 100R; PARTNO (none) -> 311-100HRCT-ND
- R32: PARTNO (none) -> RHM10.0KHCT-ND
- R35: PARTNO (none) -> 311-120GRCT-ND
- U$1, U$2, U$3, U$4, U$5, U$6: PARTNO (none) -> IRFS7530-7PPBF-ND
- U$10: PARTNO (none) -> MAX6103EUR+TCT-ND
- U$11: PARTNO (none) -> 490-4800-1-ND
- U$12: PARTNO (none) -> 553-2258-ND
- U$7, U$8: PARTNO (none) -> WSLR-.0003CT-ND
- U$9: PARTNO (none) -> 296-29433-1-ND
- U1: PARTNO (none) -> MCP2551T-E/SNCT-ND
- X1: DIGIKEY 535-9721-2-ND -> (none); PARTNO (none) -> 535-9721-1-ND
Connections:
- removed net VSS1: C41.2, C42.2, IC1.VSS1, IC1.VSS4
- removed net VSSA: C36.2, IC1.VSSA
- new net N$34: D6.C, R37.2
- net AGND: now also PT1.P$2
- net GH_A: no longer TP1.TP
- net GH_B: no longer TP4.TP
- net GH_C: no longer TP7.TP
- net GND: now also C36.2, C41.2, C42.2, C49.2, C50.2, C51.2, IC1.VSS1, IC1.VSS4, IC1.VSSA, PT1.P$1, R37.1; no longer U$9.PVDD2_1, U$9.PVDD2_2
- net M_A: no longer TP2.TP
- net M_B: no longer TP5.TP
- net M_C: no longer TP8.TP
- net SN1: no longer TP10.TP
- net SN2: no longer TP12.TP
- net VCC: now also D6.A
- net VDD: now also U$9.PVDD2_1, U$9.PVDD2_2
- net VSENS_A: now also C49.1
- net VSENS_B: now also C50.1
- net VSENS_C: now also C51.1
Other:
- moved on the sheet: C18, R26, R27, R30, R31, TP34, TP35, TP36
